Commit message: Added centre of mass codegen and task

File: examples/cassie/model/urdf/cassie.urdf (robot description, URDF)
Before this commit: robot cassie, 18 links, 17 joints
Links:
- removed link base_link
Joints:
- removed joint base_joint

Commit message: WIP: adding full state, encountered issues. Notes in codegen.cc

File: examples/cassie/model/urdf/cassie.urdf (robot description, URDF)
Before this commit: robot cassie, 17 links, 16 joints
Links:
- added link base_link, mass 0.000001
Joints:
- added joint base_joint: type floating, parent base_link, child pelvis, origin xyz=0 0 0 rpy=0 0 0

Commit message: Fixed contact locations by adding these frames to the URDF file. The way pinocchio handles fixed frames does not work well with our current set up, so the set-up has been changed to only compute end-effector data for frames that already exist in the system, not ones that you can add arbitrarily. This may need to be reconsidered later on but for now we have the correct contact locations (also avoided using the transforms from the wiki and instead found the locations of these points in the ankle frame from the cassierl github)

File: examples/cassie/model/urdf/cassie.urdf (robot description, URDF)
Before this commit: robot cassie, 18 links, 17 joints
Links:
- added link leftfootback
- added link leftfootfront
- added link rightfootback
- added link rightfootfront
Joints:
- added joint LeftFootBack: type fixed, parent leftfoot, child leftfootback, origin xyz=0.08 0.005 0
- added joint LeftFootFront: type fixed, parent leftfoot, child leftfootfront, origin xyz=-0.0407 0.107 0
- added joint RightFootBack: type fixed, parent rightfoot, child rightfootback, origin xyz=0.08 0.005 0
- added joint RightFootFront: type fixed, parent rightfoot, child rightfootfront, origin xyz=-0.0407 0.107 0
