Commit message: Testing on fully actuated arm for tasks and joint tracking, appears to work well, confirming correct implementation of tasks. Further work on Cassie leg required to get similar goal achieved, will test arm with holonomic constraints added and gearing in the next commit

File: examples/arm/model/urdf/arm.urdf (robot description, URDF)
Before this commit: robot arm, 5 links, 4 joints
Links:
- link first_link: geometry visual cylinder length=1.0 radius=0.05
- link second_link: mass 0.3 -> 1.0; geometry visual cylinder length=1.0 radius=0.05
- link third_link: mass 0.3 -> 1.3; geometry visual cylinder length=1.0 radius=0.05
Joints:
- removed joint third_joint
- added joint wrist: type revolute, parent second_link, child third_link, origin xyz=0 0 -1.0 rpy=0 0 0, axis 1 0 0, limit lower=-3.1415 upper=3.1415 effort=100.0 velocity=5
- joint base_joint: origin xyz=0 0 0 rpy=0 0 0 -> xyz=0 0 2.5 rpy=0 0 0
- joint elbow: limit lower=-2.0857 upper=2.0857 effort=100.0 velocity=5 -> lower=-3.1415 upper=3.1415 effort=100.0 velocity=5
- joint shoulder: limit lower=-2.0857 upper=2.0857 effort=100.0 velocity=5 -> lower=-3.1415 upper=3.1415 effort=100.0 velocity=5; type prismatic -> revolute

Commit message: Arm updates for trial test, working on making codegeneration functions translatable to other libraries, working on adding holonomic constraints to OSC in a different way with the option of explicitly or implicitly working out their constraint forces

File: examples/arm/model/urdf/arm.urdf (robot description, URDF)
Before this commit: robot arm, 5 links, 4 joints
Links:
- removed link base
- link first_link: mass 1 -> 1.0
- link third_link: mass 1.3 -> 1.0
Joints:
- removed joint base_joint
- joint shoulder: parent base -> base_link

Commit message: Changed cassie_fixed and arm experiments to new reference frame config

File: examples/arm/model/urdf/arm.urdf (robot description, URDF)
Before this commit: robot arm, 4 links, 3 joints
Links:
- added link hand_frame
Joints:
- added joint hand: type fixed, parent third_link, child hand_frame, origin xyz=0 0 -1.0 rpy=0 0 0
